Commit message: URDF model of first robot. Contains most of the geometry, including kinect/US sensors

File: URDF-models/adam.urdf (robot description, URDF)
Before this commit: robot ADAM, 10 links, 9 joints
Links:
- added link castor_pivot; visual cylinder length=0.005 radius=0.015
- added link castor_wheel; visual cylinder length=0.014 radius=0.015
- added link front_center_ultrasonic_sensor; visual mesh filename=file:///home/brian/robotics_code/ROS/URDF-models/ultrasonic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
- added link front_left_ultrasonic_sensor; visual mesh filename=file:///home/brian/robotics_code/ROS/URDF-models/ultrasonic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
- added link front_right_ultrasonic_sensor; visual mesh filename=file:///home/brian/robotics_code/ROS/URDF-models/ultrasonic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
- added link kinect; visual mesh filename=file:///home/brian/robotics_code/ROS/URDF-models/kinect.dae
- added link rear_center_ultrasonic_sensor; visual mesh filename=file:///home/brian/robotics_code/ROS/URDF-models/ultrasonic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
- added link rear_left_ultrasonic_sensor; visual mesh filename=file:///home/brian/robotics_code/ROS/URDF-models/ultrasonic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
- added link rear_right_ultrasonic_sensor; visual mesh filename=file:///home/brian/robotics_code/ROS/URDF-models/ultrasonic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
Joints:
- added joint base_to_caster_pivot: type continuous, parent base_link, child castor_pivot, origin xyz=0 -0.19 -0.0115, axis 0 0 1
- added joint base_to_front_center_ultrasonic_sensor: type fixed, parent base_link, child front_center_ultrasonic_sensor, origin xyz=0 0 0 rpy=0 0 0
- added joint base_to_front_left_ultrasonic_sensor: type fixed, parent base_link, child front_left_ultrasonic_sensor, origin xyz=-0.09 0 0 rpy=0 0 0.523
- added joint base_to_front_right_ultrasonic_sensor: type fixed, parent base_link, child front_right_ultrasonic_sensor, origin xyz=0.09 0 0 rpy=0 0 -0.523
- added joint base_to_kinect: type fixed, parent base_link, child kinect, origin xyz=0 -.05 .10 rpy=0 0 3.141593
- added joint base_to_rear_center_ultrasonic_sensor: type fixed, parent base_link, child rear_center_ultrasonic_sensor, origin xyz=0 -0.20 0 rpy=0 0 3.1415
- added joint base_to_rear_left_ultrasonic_sensor: type fixed, parent base_link, child rear_left_ultrasonic_sensor, origin xyz=-0.06 -0.16 0 rpy=0 0 2.36
- added joint base_to_rear_right_ultrasonic_sensor: type fixed, parent base_link, child rear_right_ultrasonic_sensor, origin xyz=0.06 -0.16 0 rpy=0 0 -2.36
- added joint caster_pivot_to_caster_wheel: type continuous, parent castor_pivot, child castor_wheel, origin xyz=0 -0.012 -0.02 rpy=0 1.57075 0, axis 0 0 1
