Commit message: Reorganized robot description

File: ADAM_description/model.urdf (robot description, URDF)
Before this commit: robot ADAM, 19 links, 18 joints
Links:
- link base_link: geometry visual mesh filename=file:///home/brian/robotics_code/ROS/ADAM_description/meshe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
- link front_center_ultrasonic_sensor: geometry visual mesh filename=file:///home/brian/robotics_code/ROS/ADAM_description/meshe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
- link front_left_ultrasonic_sensor: geometry visual mesh filename=file:///home/brian/robotics_code/ROS/ADAM_description/meshe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
- link front_right_ultrasonic_sensor: geometry visual mesh filename=file:///home/brian/robotics_code/ROS/ADAM_description/meshe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
- link kinect: geometry visual mesh filename=file:///home/brian/robotics_code/ROS/ADAM_description/meshe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
- link left_wheel: geometry visual mesh filename=file:///home/brian/robotics_code/ROS/ADAM_description/meshe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
- link rear_center_ultrasonic_sensor: geometry visual mesh filename=file:///home/brian/robotics_code/ROS/ADAM_description/meshe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
- link rear_left_ultrasonic_sensor: geometry visual mesh filename=file:///./meshes/ultrasonic_sensor_with_mount.dae
- link rear_right_ultrasonic_sensor: geometry visual mesh filename=file:///home/brian/robotics_code/ROS/ADAM_description/meshe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
- link right_wheel: geometry visual mesh filename=file:///home/brian/robotics_code/ROS/ADAM_description/meshe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

Commit message: Added dummy inertial info to robot URDF so that I can get it into gazebo

File: ADAM_description/model.urdf (robot description, URDF)
Before this commit: robot ADAM, 19 links, 18 joints
Links:
- link base_link: mass None -> 1
- link castor_pivot: mass None -> 1
- link castor_wheel: mass None -> 1
- link drawer: mass None -> 1
- link front_center_ultrasonic_sensor: mass None -> 1
- link front_left_ultrasonic_sensor: mass None -> 1
- link front_right_ultrasonic_sensor: mass None -> 1
- link kinect: mass None -> 1
- link left_axle: mass None -> 1
- link left_motor: mass None -> 1
- link left_riser_level1: mass None -> 1
- link left_wheel: mass None -> 1
- link rear_center_ultrasonic_sensor: mass None -> 1
- link rear_left_ultrasonic_sensor: mass None -> 1; geometry visual mesh filename=file:///home/brian/robotics_code/ROS/ADAM_description/meshe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
- link rear_right_ultrasonic_sensor: mass None -> 1
- link right_axle: mass None -> 1
- link right_motor: mass None -> 1
- link right_riser_level1: mass None -> 1
- link right_wheel: mass None -> 1
