Commit message: URDF model that can be seen in gazebo. Start gazebo with 'roslaunch gazebo_ros empty_world.launch' and launch model with 'rosrun gazebo_ros spawn_model -file /home/brian/robotics_code/ROS/workspace/src/adam_description/urdf/adam.urdf -urdf -model adam'

File: workspace/src/adam_description/urdf/adam.urdf (robot description, URDF)
Before this commit: robot ADAM, 19 links, 18 joints
Links:
- link base_link: geometry collision mesh filename=package://adam_description/meshes/adam_base.dae; visual mesh filename=package://adam_description/meshes/adam_base.dae
- link front_center_ultrasonic_sensor: geometry visual mesh filename=package://adam_description/meshes/ultrasonic_sensor_with_mo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
- link front_left_ultrasonic_sensor: geometry visual mesh filename=package://adam_description/meshes/ultrasonic_sensor_with_mo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
- link front_right_ultrasonic_sensor: geometry visual mesh filename=package://adam_description/meshes/ultrasonic_sensor_with_mo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
- link kinect: geometry visual mesh filename=package://adam_description/meshes/kinect.dae
- link left_wheel: geometry visual mesh filename=package://adam_description/meshes/wheel_90mm.dae
- link rear_center_ultrasonic_sensor: geometry visual mesh filename=package://adam_description/meshes/ultrasonic_sensor_with_mo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
- link rear_left_ultrasonic_sensor: geometry visual mesh filename=package://adam_description/meshes/ultrasonic_sensor_with_mo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
- link rear_right_ultrasonic_sensor: geometry visual mesh filename=package://adam_description/meshes/ultrasonic_sensor_with_mo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
- link right_wheel: geometry visual mesh filename=package://adam_description/meshes/wheel_90mm.dae

Commit message: Added collision properties to wheels

File: workspace/src/adam_description/urdf/adam.urdf (robot description, URDF)
Before this commit: robot ADAM, 19 links, 18 joints
Links:
- link castor_wheel: geometry collision cylinder length=0.014 radius=0.015; visual cylinder length=0.014 radius=0.015
- link left_wheel: geometry collision mesh filename=package://adam_description/meshes/wheel_90mm.dae; visual mesh filename=package://adam_description/meshes/wheel_90mm.dae
- link right_wheel: geometry collision mesh filename=package://adam_description/meshes/wheel_90mm.dae; visual mesh filename=package://adam_description/meshes/wheel_90mm.dae

Commit message: new robot description (mostly finished) and launch file for viz

File: workspace/src/adam_description/urdf/adam.urdf (robot description, URDF)
Before this commit: robot ADAM, 19 links, 18 joints
Links:
- removed link castor_pivot
- removed link castor_wheel
- removed link drawer
- removed link front_center_ultrasonic_sensor
- removed link front_left_ultrasonic_sensor
- removed link front_right_ultrasonic_sensor
- removed link kinect
- removed link left_riser_level1
- removed link left_wheel
- removed link rear_center_ultrasonic_sensor
- removed link rear_left_ultrasonic_sensor
- removed link rear_right_ultrasonic_sensor
- removed link right_riser_level1
- removed link right_wheel
- added link black_plastic_base; visual box size=0.16 0.2 ${black_plastic_thickness}
- added link left_active_wheel; visual cylinder length=0.008 radius=0.0325
- added link left_base; visual box size=0.29 ${channel_width} ${channel_width}
- added link rear_base; visual box size=0.16 ${channel_width} ${channel_width}
- added link right_active_wheel; visual cylinder length=0.008 radius=0.0325
- added link right_base; visual box size=0.29 ${channel_width} ${channel_width}
- link base_link: mass 1 -> None; geometry visual box size=0.16 ${channel_width} ${channel_width}
- link left_axle: mass 1 -> None; geometry visual cylinder length=${axle_length} radius=0.0025
- link left_motor: mass 1 -> None; geometry visual cylinder length=${motor_length} radius=${motor_radius}
- link right_axle: mass 1 -> None; geometry visual cylinder length=${axle_length} radius=0.0025
- link right_motor: mass 1 -> None; geometry visual cylinder length=0.065 radius=0.02
Joints:
- removed joint base_to_caster_pivot
- removed joint base_to_drawer
- removed joint base_to_front_center_ultrasonic_sensor
- removed joint base_to_front_left_ultrasonic_sensor
- removed joint base_to_front_right_ultrasonic_sensor
- removed joint base_to_kinect
- removed joint base_to_left_riser_level1
- removed joint base_to_rear_center_ultrasonic_sensor
- removed joint base_to_rear_left_ultrasonic_sensor
- removed joint base_to_rear_right_ultrasonic_sensor
- removed joint base_to_right_riser_level1
- removed joint caster_pivot_to_caster_wheel
- removed joint left_wheel_to_axle
- removed joint right_wheel_to_axle
- added joint black_plastic_base_to_front_base: type fixed, parent base_link, child black_plastic_base, origin xyz=0 -0.02 ${1.5*channel_width} rpy=0 0 0, axis 0 0 0
- added joint left_active_wheel_to_axle: type fixed, parent left_axle, child left_active_wheel, origin xyz=0 0 -0.02
- added joint left_base_to_front_base: type fixed, parent base_link, child left_base, origin xyz=0.064 0 0 rpy=0 0 ${pi/2}, axis 0 0 0
- added joint rear_base_to_front_base: type fixed, parent base_link, child rear_base, origin xyz=0 -0.1 ${channel_width} rpy=0 0 0, axis 0 0 0
- added joint right_active_wheel_to_axle: type fixed, parent right_axle, child right_active_wheel, origin xyz=0 0 0.02
- added joint right_base_to_front_base: type fixed, parent base_link, child right_base, origin xyz=-0.064 0 0 rpy=0 0 ${pi/2}, axis 0 0 0
- joint left_axle_to_motor: axis 0 0 1 -> (none); origin xyz=0.0 0 0.045 rpy=0 0 0 -> xyz=0 0 ${-motor_length/2}
- joint left_motor_to_base: origin xyz=-0.075 0 -.03 rpy=0 -1.57075 0 -> xyz=-0.045 0 ${1.5*channel_width + black_plastic_thickness + 0.021} rpy=0 1.57075 0
- joint right_axle_to_motor: axis 0 0 1 -> (none); origin xyz=0.0 0 0.045 rpy=0 0 0 -> xyz=0 0 ${motor_length/2}
- joint right_motor_to_base: origin xyz=0.075 0 -.03 rpy=0 1.57075 0 -> xyz=0.045 0 ${1.5*channel_width + black_plastic_thickness + 0.021} rpy=0 1.57075 0

Commit message: add kinect to adam urdf

File: workspace/src/adam_description/urdf/adam.urdf (robot description, URDF)
Before this commit: robot ADAM, 11 links, 10 joints
Links:
- added link kinect; collision mesh filename=package://adam_description/meshes/kinect.dae; visual mesh filename=package://adam_description/meshes/kinect.dae
Joints:
- added joint kinet_to_base: type fixed, parent base_link, child kinect, origin xyz=0 0 0.2 rpy=0 0 0, axis 0 0 0

Commit message: correct orientation of kinect sensor, show registered point cloud in rviz

File: workspace/src/adam_description/urdf/adam.urdf (robot description, URDF)
Before this commit: robot ADAM, 12 links, 11 joints
Links:
- added link kinect_sensor
Joints:
- removed joint kinet_to_base
- added joint kinect_sensor_to_kinect: type fixed, parent kinect, child kinect_sensor, origin xyz=0 0 0 rpy=1.57075 3.14159 0
- added joint kinect_to_base: type fixed, parent base_link, child kinect, origin xyz=0 0 0.2 rpy=0 0 0, axis 0 0 0
